Commit message: same simulation environment done

File: robot_description/Ground/magneto/ground_3d.urdf (robot description, URDF)
Before this commit: robot ground_skeleton, 4 links, 3 joints
Links:
- link wall_link: geometry collision box size=50.0 50.0 2.3; visual mesh filename=mesh/tile_marble_diamond.dae scale=1. 1. 0.1

File: robot_description/Ground/magneto/ground_climbing.urdf (robot description, URDF)
Before this commit: robot ground_skeleton, 3 links, 2 joints
Links:
- link ground_link: geometry collision box size=5000.0 500.0 0.05; visual mesh filename=mesh/tile_marble_diamond.dae scale=1. 1. 1.
- link wall_link: geometry collision box size=50.0 50.0 2.3; visual mesh filename=mesh/tile_marble_diamond.dae scale=1. 1. 1.

File: robot_description/Ground/magneto/ground_inclined.urdf (robot description, URDF)
Before this commit: robot ground_skeleton, 3 links, 2 joints
Links:
- link ground_link: geometry collision box size=5000.0 500.0 0.05; visual mesh filename=mesh/tile_marble_diamond.dae scale=1. 1. 0.1
- link wall_link: geometry collision box size=50.0 50.0 2.3; visual mesh filename=mesh/tile_marble_diamond.dae scale=1. 1. 0.1

File: robot_description/Ground/magneto/ground_inclined02.urdf (robot description, URDF)
Before this commit: robot ground_skeleton, 3 links, 2 joints
Links:
- link ground_link: geometry collision box size=5000.0 500.0 0.05; visual mesh filename=mesh/tile_marble_diamond.dae scale=1. 1. 0.1
- link wall_link: geometry collision box size=50.0 50.0 2.3; visual mesh filename=mesh/tile_marble_diamond.dae scale=1. 1. 0.1

File: robot_description/Ground/magneto/ground_inclined04.urdf (robot description, URDF)
Before this commit: robot ground_skeleton, 3 links, 2 joints
Links:
- link ground_link: geometry collision box size=5000.0 500.0 0.05; visual mesh filename=mesh/tile_marble_diamond.dae scale=1. 1. 0.1
- link wall_link: geometry collision box size=50.0 50.0 2.3; visual mesh filename=mesh/tile_marble_diamond.dae scale=1. 1. 0.1

File: robot_description/Ground/magneto/wall.urdf (robot description, URDF)
Before this commit: robot ground_skeleton, 4 links, 3 joints
Links:
- removed link world_frame
- link ground_link: geometry collision box size=500.0 500.0 0.05; visual mesh filename=mesh/tile_marble_diamond.dae scale=0.1 0.1 0.01
- link wall_link: geometry collision box size=2.0 2.0 0.01; visual box size=2.0 2.0 0.01
Joints:
- removed joint frame_joint
- joint ground_joint: origin xyz=0 0 -0.01 rpy=0 1 0 -> xyz=0 0 0 rpy=0 0 0
- joint wall_joint: origin xyz=4 -10 -10 rpy=0 -1.5708 0 -> xyz=0 1 1 rpy=0 -1.5708 0; parent world -> ground_link
