Commit message: fixed state_estimator init, still not working

File: robot_description/Ground/magneto/wall.urdf (robot description, URDF)
Before this commit: robot ground_skeleton, 3 links, 2 joints
Links:
- link ground_link: geometry collision box size=2.0 2.0 0.01; visual box size=2.0 2.0 0.01
Joints:
- joint ground_joint: origin xyz=0 0 0 rpy=0 0 0 -> xyz=0 0 0 rpy=0 0 3.141592
- joint wall_joint: origin xyz=0 1 1 rpy=0 -1.5708 0 -> xyz=0 1 1 rpy=0 1.5708 0
